Commit message: change base joint to floating type

File: robots_urdf/ada_with_camera.urdf (robot description, URDF)
Before this commit: robot j2n6s200, 16 links, 15 joints
Joints:
- joint j2n6s200_joint_base: type fixed -> floating

Commit message: fix finger collision check

File: robots_urdf/ada_with_camera.urdf (robot description, URDF)
Before this commit: robot j2n6s200, 16 links, 15 joints
Links:
- link j2n6s200_link_6: geometry collision mesh filename=package://ada_description/meshes/collision_hand_2finger.dae; visual mesh filename=package://ada_description/meshes/collision_hand_2finger.dae
- link j2n6s200_link_finger_1: geometry collision mesh filename=package://ada_description/meshes/finger.dae; visual mesh filename=package://ada_description/meshes/finger_proximal.dae
- link j2n6s200_link_finger_2: geometry collision mesh filename=package://ada_description/meshes/finger.dae; visual mesh filename=package://ada_description/meshes/finger_proximal.dae
